File: Eagle files/Drone.brd (EAGLE design)
At the start: 83.8 x 42.9 mm, 25 parts, among them U1 GY-521MPU6050

Commit message: Updated the Drone board files
Parts:
- moved SCL-2 7.18 mm to (90.2, 41.9)
- moved SDA-2 7.18 mm to (87.6, 41.9)
Connections:
- net SCL: now also ARDUINO_NANO.9; no longer ARDUINO_NANO.11
- net SDA: now also ARDUINO_NANO.8; no longer ARDUINO_NANO.10
Changed lines of the file:
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@@
 <hole x="95.25" y="49.53" drill="1"/>
 <hole x="92.71" y="41.91" drill="1"/>
-<hole x="90.17" y="41.91" drill="1"/>
+<hole x="92.71" y="36.83" drill="1"/>
 <hole x="90.17" y="44.45" drill="1"/>
 <hole x="90.17" y="49.53" drill="1"/>
@@
 <hole x="105.41" y="57.15" drill="1"/>
 <hole x="102.87" y="57.15" drill="1"/>
-<hole x="87.63" y="41.91" drill="1"/>
+<hole x="95.25" y="36.83" drill="1"/>
 <hole x="116.153" y="56.027" drill="3"/>
 <hole x="116.15" y="40.486" drill="3"/>
@@
 <attribute name="VALUE" x="124.46" y="48.26" size="0.0254" layer="28" rot="MR0"/>
 </element>
-<element name="SDA-2" library="wirepad" library_urn="urn:adsk.eagle:library:412" package="1,6/0,8" package3d_urn="urn:adsk.eagle:package:30830/1" value="SDA" x="92.71" y="36.83" smashed="yes" rot="MR0">
-<attribute name="POPULARITY" value="1" x="92.71" y="36.83" size="1.778" layer="28" rot="MR0" display="off"/>
-<attribute name="VALUE" x="92.71" y="37.43" size="0.0254" layer="28" rot="MR0"/>
-</element>
-<element name="SCL-2" library="wirepad" library_urn="urn:adsk.eagle:library:412" package="1,6/0,8" package3d_urn="urn:adsk.eagle:package:30830/1" value="SCL" x="95.25" y="36.83" smashed="yes" rot="MR0">
-<attribute name="POPULARITY" value="1" x="95.25" y="36.83" size="1.778" layer="28" rot="MR0" display="off"/>
-<attribute name="VALUE" x="95.25" y="37.43" size="0.0254" layer="28" rot="MR0"/>
+<element name="SDA-2" library="wirepad" library_urn="urn:adsk.eagle:library:412" package="1,6/0,8" package3d_urn="urn:adsk.eagle:package:30830/1" value="SDA" x="87.63" y="41.91" smashed="yes" rot="MR0">
+<attribute name="POPULARITY" value="1" x="87.63" y="41.91" size="1.778" layer="28" rot="MR0" display="off"/>
+<attribute name="VALUE" x="87.63" y="42.51" size="0.0254" layer="28" rot="MR0"/>
+</element>
+<element name="SCL-2" library="wirepad" library_urn="urn:adsk.eagle:library:412" package="1,6/0,8" package3d_urn="urn:adsk.eagle:package:30830/1" value="SCL" x="90.17" y="41.91" smashed="yes" rot="MR0">
+<attribute name="POPULARITY" value="1" x="90.17" y="41.91" size="1.778" layer="28" rot="MR0" display="off"/>
+<attribute name="VALUE" x="90.17" y="42.51" size="0.0254" layer="28" rot="MR0"/>
 </element>
 <element name="VCC-1" library="wirepad" library_urn="urn:adsk.eagle:library:412" package="1,6/0,8" package3d_urn="urn:adsk.eagle:package:30830/1" value="VCC" x="82.55" y="62.23" smashed="yes" rot="MR0">
@@
 <wire x1="128.07" y1="44.45" x2="125.73" y2="44.45" width="0.8128" layer="16"/>
 <contactref element="U1" pad="SCL"/>
-<contactref element="ARDUINO_NANO" pad="11"/>
+<contactref element="ARDUINO_NANO" pad="9"/>
 <contactref element="SCL-2" pad="1"/>
-<wire x1="95.25" y1="36.83" x2="95.25" y2="39.37" width="0.8128" layer="16"/>
-<wire x1="95.25" y1="39.37" x2="125.73" y2="44.45" width="0" layer="19" extent="1-1"/>
+<wire x1="90.17" y1="41.91" x2="90.17" y2="39.37" width="0.8128" layer="16"/>
+<wire x1="90.17" y1="41.91" x2="125.73" y2="44.45" width="0" layer="19" extent="1-1"/>
 </signal>
 <signal name="SDA">
 <contactref element="SDA" pad="1"/>
 <contactref element="U1" pad="SDA"/>
-<contactref element="ARDUINO_NANO" pad="10"/>
-<contactref element="SDA-2" pad="1"/>
 <wire x1="128.109996875" y1="46.75680625" x2="128.048778125" y2="46.99" width="0.8128" layer="16"/>
 <wire x1="125.73" y1="46.99" x2="128.048778125" y2="46.99" width="0.8128" layer="16"/>
-<wire x1="92.71" y1="36.83" x2="92.71" y2="39.37" width="0.8128" layer="16"/>
-<wire x1="92.71" y1="39.37" x2="125.73" y2="46.99" width="0" layer="19" extent="1-1"/>
+<contactref element="ARDUINO_NANO" pad="8"/>
+<contactref element="SDA-2" pad="1"/>
+<wire x1="87.63" y1="41.91" x2="87.63" y2="39.37" width="0.8128" layer="16"/>
+<wire x1="128.109996875" y1="46.75680625" x2="128.11" y2="46.99" width="0" layer="19" extent="16-16"/>
+<wire x1="87.63" y1="41.91" x2="125.73" y2="46.99" width="0" layer="19" extent="1-1"/>
 </signal>
 <signal name="ESC3">
