File: Eagle files/Drone.sch (EAGLE design)
At the start: 25 parts, among them U1 GY-521MPU6050

Commit message: Updated the Drone board files
Connections:
- net SCL: now also ARDUINO_NANO.A5; no longer ARDUINO_NANO.A7
- net SDA: now also ARDUINO_NANO.A4; no longer ARDUINO_NANO.A6
Changed lines of the file:
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@@
 <instance part="SCL" gate="G$1" x="20.32" y="96.52" smashed="yes" rot="R90"/>
 <instance part="SDA" gate="G$1" x="25.4" y="96.52" smashed="yes" rot="R90"/>
-<instance part="SDA-2" gate="G$1" x="58.42" y="55.88" smashed="yes" rot="R180"/>
-<instance part="SCL-2" gate="G$1" x="58.42" y="58.42" smashed="yes" rot="R180"/>
+<instance part="SDA-2" gate="G$1" x="55.88" y="50.8" smashed="yes" rot="R180"/>
+<instance part="SCL-2" gate="G$1" x="55.88" y="53.34" smashed="yes" rot="R180"/>
 <instance part="VCC-1" gate="G$1" x="-35.56" y="78.74" smashed="yes" rot="R270"/>
 <instance part="VCC-2" gate="G$1" x="53.34" y="68.58" smashed="yes" rot="R180"/>
@@
 </segment>
 <segment>
-<pinref part="ARDUINO_NANO" gate="G$1" pin="A7"/>
+<pinref part="ARDUINO_NANO" gate="G$1" pin="A5"/>
+<wire x1="48.26" y1="53.34" x2="53.34" y2="53.34" width="0.1524" layer="91"/>
 <pinref part="SCL-2" gate="G$1" pin="P"/>
-<wire x1="48.26" y1="58.42" x2="55.88" y2="58.42" width="0.1524" layer="91"/>
-<label x="60.96" y="58.42" size="1.778" layer="95"/>
+<label x="58.42" y="53.34" size="1.778" layer="95"/>
 </segment>
 </net>
@@
 </segment>
 <segment>
-<pinref part="ARDUINO_NANO" gate="G$1" pin="A6"/>
+<pinref part="ARDUINO_NANO" gate="G$1" pin="A4"/>
+<wire x1="48.26" y1="50.8" x2="53.34" y2="50.8" width="0.1524" layer="91"/>
 <pinref part="SDA-2" gate="G$1" pin="P"/>
-<wire x1="48.26" y1="55.88" x2="55.88" y2="55.88" width="0.1524" layer="91"/>
-<label x="60.96" y="55.88" size="1.778" layer="95"/>
+<label x="58.42" y="50.8" size="1.778" layer="95"/>
 </segment>
 </net>
